Commit message: Sync for release v1.8.330

File: ros2/src/rbq_description/urdf/rbq.urdf (robot description, URDF)
Before this commit: robot rbq10, 18 links, 17 joints
Joints:
- joint imu_joint: child trunk -> imu_link; origin xyz=-0.00665 0 0.0404 rpy=0 0 0 -> xyz=0.00665 0 -0.0404 rpy=0 0 0; parent imu_link -> trunk
