Commit message: Sync for release v1.11.21

File: resources/urdf/rbq10.urdf (robot description, URDF)
Before this commit: robot rbq10, 17 links, 16 joints
Links:
- link FL_foot: geometry collision sphere radius=0.03; visual sphere radius=0.001
- link FR_foot: geometry collision sphere radius=0.03; visual sphere radius=0.001
- link HL_foot: geometry collision sphere radius=0.03; visual sphere radius=0.001
- link HR_foot: geometry collision sphere radius=0.03; visual sphere radius=0.001
